Commit message: cambios en orientacion de lidar y nodo

File: src/puzzlebot_gazebo/urdf/puzzlebot.xacro (robot description, xacro)
@@ -218,5 +218,5 @@
         <parent link="chassis"/>
         <child link="lidar"/>
-        <origin xyz="0.05 0 0.115" rpy="0 0 ${PI}"/>
+        <origin xyz="0.05 0 0.115" rpy="0 0 0"/>
     </joint>
 	<!-- TRANSMISSIONS (For a more complex model and it represents actuator attributes) -->
